Commit message: URDF, xaco 수정

File: src/quattro_description/urdf/quattro.urdf (robot description, URDF)
Before this commit: robot quattro, 17 links, 16 joints
Joints:
- joint back_left_hip_joint: limit lower=-1.04 upper=1.04 effort=40.0 velocity=4.0 -> lower=-0.7853981634 upper=0.7853981634 effort=11.0 velocity=12.5663706144
- joint back_left_lower_leg_joint: limit lower=-2.4783675378 upper=2.4783675378 effort=40.0 velocity=4.0 -> lower=-2.3561944902 upper=2.3561944902 effort=11.0 velocity=12.5663706144
- joint back_left_upper_leg_joint: limit lower=-1.57079632679 upper=2.59 effort=40.0 velocity=4.0 -> lower=-1.5707963268 upper=2.4434609528 effort=11.0 velocity=12.5663706144
- joint back_right_hip_joint: limit lower=-1.04 upper=1.04 effort=40.0 velocity=4.0 -> lower=-0.7853981634 upper=0.7853981634 effort=11.0 velocity=12.5663706144
- joint back_right_lower_leg_joint: limit lower=-2.4783675378 upper=2.4783675378 effort=40.0 velocity=4.0 -> lower=-2.3561944902 upper=2.3561944902 effort=11.0 velocity=12.5663706144
- joint back_right_upper_leg_joint: limit lower=-1.57079632679 upper=2.59 effort=40.0 velocity=4.0 -> lower=-1.5707963268 upper=2.4434609528 effort=11.0 velocity=12.5663706144
- joint front_left_hip_joint: limit lower=-1.04 upper=1.04 effort=40.0 velocity=4.0 -> lower=-0.7853981634 upper=0.7853981634 effort=11.0 velocity=12.5663706144
- joint front_left_lower_leg_joint: limit lower=-2.4783675378 upper=2.4783675378 effort=40.0 velocity=4.0 -> lower=-2.3561944902 upper=2.3561944902 effort=11.0 velocity=12.5663706144
- joint front_left_upper_leg_joint: limit lower=-1.57079632679 upper=2.59 effort=40.0 velocity=4.0 -> lower=-1.5707963268 upper=2.4434609528 effort=11.0 velocity=12.5663706144
- joint front_right_hip_joint: limit lower=-1.04 upper=1.04 effort=40.0 velocity=4.0 -> lower=-0.7853981634 upper=0.7853981634 effort=11.0 velocity=12.5663706144
- joint front_right_lower_leg_joint: limit lower=-2.4783675378 upper=2.4783675378 effort=40.0 velocity=4.0 -> lower=-2.3561944902 upper=2.3561944902 effort=11.0 velocity=12.5663706144
- joint front_right_upper_leg_joint: limit lower=-1.57079632679 upper=2.59 effort=40.0 velocity=4.0 -> lower=-1.5707963268 upper=2.4434609528 effort=11.0 velocity=12.5663706144

File: src/quattro_description/urdf/quattro.urdf.xacro (robot description, xacro)
@@ -142,6 +142,8 @@
     <child link="front_left_hip_link"/>
     <axis xyz="1 0 0"/>
-    <limit lower="-1.04" upper="1.04" effort="40.0" velocity="4.0"/>
-    <dynamics damping="0.0" friction="0.0"/>
+    <!-- hip joint limit: -45~45 deg | effort: stall torque 11N·m, velocity: rated speed 120rpm = 12.5663706144 rad/s (motor: 6010-8) -->
+    <limit lower="-0.7853981634" upper="0.7853981634" effort="11.0" velocity="12.5663706144"/>
+    <!-- friction: no-load current 0.4A x torque constant 0.47N·m/A = 0.188N·m (Coulomb friction estimate); damping: not given in datasheet, kept at 0.0 -->
+    <dynamics damping="0.0" friction="0.188"/>
   </joint>
   <link name="front_left_upper_leg_link">
@@ -165,6 +167,8 @@
     <child link="front_left_upper_leg_link"/>
     <axis xyz="0 1 0"/>
-    <limit lower="-1.57079632679" upper="2.59" effort="40.0" velocity="4.0"/>
-    <dynamics damping="0.0" friction="0.0"/>
+    <!-- upper joint limit: -90~140 deg | effort: stall torque 11N·m, velocity: rated speed 120rpm = 12.5663706144 rad/s (motor: 6010-8) -->
+    <limit lower="-1.5707963268" upper="2.4434609528" effort="11.0" velocity="12.5663706144"/>
+    <!-- friction: no-load current 0.4A x torque constant 0.47N·m/A = 0.188N·m (Coulomb friction estimate); damping: not given in datasheet, kept at 0.0 -->
+    <dynamics damping="0.0" friction="0.188"/>
   </joint>
   <link name="front_left_lower_leg_link">
@@ -188,6 +192,8 @@
     <child link="front_left_lower_leg_link"/>
     <axis xyz="0 1 0"/>
-    <limit lower="-2.4783675378" upper="2.4783675378" effort="40.0" velocity="4.0"/>
-    <dynamics damping="0.0" friction="0.0"/>
+    <!-- lower joint limit: -135~135 deg | effort: stall torque 11N·m, velocity: rated speed 120rpm = 12.5663706144 rad/s (motor: 6010-8) -->
+    <limit lower="-2.3561944902" upper="2.3561944902" effort="11.0" velocity="12.5663706144"/>
+    <!-- friction: no-load current 0.4A x torque constant 0.47N·m/A = 0.188N·m (Coulomb friction estimate); damping: not given in datasheet, kept at 0.0 -->
+    <dynamics damping="0.0" friction="0.188"/>
   </joint>
   <link name="front_left_foot_link">
@@ -240,6 +246,8 @@
     <child link="front_right_hip_link"/>
     <axis xyz="1 0 0"/>
-    <limit lower="-1.04" upper="1.04" effort="40.0" velocity="4.0"/>
-    <dynamics damping="0.0" friction="0.0"/>
+    <!-- hip joint limit: -45~45 deg | effort: stall torque 11N·m, velocity: rated speed 120rpm = 12.5663706144 rad/s (motor: 6010-8) -->
+    <limit lower="-0.7853981634" upper="0.7853981634" effort="11.0" velocity="12.5663706144"/>
+    <!-- friction: no-load current 0.4A x torque constant 0.47N·m/A = 0.188N·m (Coulomb friction estimate); damping: not given in datasheet, kept at 0.0 -->
+    <dynamics damping="0.0" friction="0.188"/>
   </joint>
   <link name="front_right_upper_leg_link">
@@ -263,6 +271,8 @@
     <child link="front_right_upper_leg_link"/>
     <axis xyz="0 1 0"/>
-    <limit lower="-1.57079632679" upper="2.59" effort="40.0" velocity="4.0"/>
-    <dynamics damping="0.0" friction="0.0"/>
+    <!-- upper joint limit: -90~140 deg | effort: stall torque 11N·m, velocity: rated speed 120rpm = 12.5663706144 rad/s (motor: 6010-8) -->
+    <limit lower="-1.5707963268" upper="2.4434609528" effort="11.0" velocity="12.5663706144"/>
+    <!-- friction: no-load current 0.4A x torque constant 0.47N·m/A = 0.188N·m (Coulomb friction estimate); damping: not given in datasheet, kept at 0.0 -->
+    <dynamics damping="0.0" friction="0.188"/>
   </joint>
   <link name="front_right_lower_leg_link">
@@ -286,6 +296,8 @@
     <child link="front_right_lower_leg_link"/>
     <axis xyz="0 1 0"/>
-    <limit lower="-2.4783675378" upper="2.4783675378" effort="40.0" velocity="4.0"/>
-    <dynamics damping="0.0" friction="0.0"/>
+    <!-- lower joint limit: -135~135 deg | effort: stall torque 11N·m, velocity: rated speed 120rpm = 12.5663706144 rad/s (motor: 6010-8) -->
+    <limit lower="-2.3561944902" upper="2.3561944902" effort="11.0" velocity="12.5663706144"/>
+    <!-- friction: no-load current 0.4A x torque constant 0.47N·m/A = 0.188N·m (Coulomb friction estimate); damping: not given in datasheet, kept at 0.0 -->
+    <dynamics damping="0.0" friction="0.188"/>
   </joint>
   <link name="front_right_foot_link">
@@ -338,6 +350,8 @@
     <child link="back_left_hip_link"/>
     <axis xyz="1 0 0"/>
-    <limit lower="-1.04" upper="1.04" effort="40.0" velocity="4.0"/>
-    <dynamics damping="0.0" friction="0.0"/>
+    <!-- hip joint limit: -45~45 deg | effort: stall torque 11N·m, velocity: rated speed 120rpm = 12.5663706144 rad/s (motor: 6010-8) -->
+    <limit lower="-0.7853981634" upper="0.7853981634" effort="11.0" velocity="12.5663706144"/>
+    <!-- friction: no-load current 0.4A x torque constant 0.47N·m/A = 0.188N·m (Coulomb friction estimate); damping: not given in datasheet, kept at 0.0 -->
+    <dynamics damping="0.0" friction="0.188"/>
   </joint>
   <link name="back_left_upper_leg_link">
@@ -361,6 +375,8 @@
     <child link="back_left_upper_leg_link"/>
     <axis xyz="0 1 0"/>
-    <limit lower="-1.57079632679" upper="2.59" effort="40.0" velocity="4.0"/>
-    <dynamics damping="0.0" friction="0.0"/>
+    <!-- upper joint limit: -90~140 deg | effort: stall torque 11N·m, velocity: rated speed 120rpm = 12.5663706144 rad/s (motor: 6010-8) -->
+    <limit lower="-1.5707963268" upper="2.4434609528" effort="11.0" velocity="12.5663706144"/>
+    <!-- friction: no-load current 0.4A x torque constant 0.47N·m/A = 0.188N·m (Coulomb friction estimate); damping: not given in datasheet, kept at 0.0 -->
+    <dynamics damping="0.0" friction="0.188"/>
   </joint>
   <link name="back_left_lower_leg_link">
@@ -384,6 +400,8 @@
     <child link="back_left_lower_leg_link"/>
     <axis xyz="0 1 0"/>
-    <limit lower="-2.4783675378" upper="2.4783675378" effort="40.0" velocity="4.0"/>
-    <dynamics damping="0.0" friction="0.0"/>
+    <!-- lower joint limit: -135~135 deg | effort: stall torque 11N·m, velocity: rated speed 120rpm = 12.5663706144 rad/s (motor: 6010-8) -->
+    <limit lower="-2.3561944902" upper="2.3561944902" effort="11.0" velocity="12.5663706144"/>
+    <!-- friction: no-load current 0.4A x torque constant 0.47N·m/A = 0.188N·m (Coulomb friction estimate); damping: not given in datasheet, kept at 0.0 -->
+    <dynamics damping="0.0" friction="0.188"/>
   </joint>
   <link name="back_left_foot_link">
@@ -436,6 +454,8 @@
     <child link="back_right_hip_link"/>
     <axis xyz="1 0 0"/>
-    <limit lower="-1.04" upper="1.04" effort="40.0" velocity="4.0"/>
-    <dynamics damping="0.0" friction="0.0"/>
+    <!-- hip joint limit: -45~45 deg | effort: stall torque 11N·m, velocity: rated speed 120rpm = 12.5663706144 rad/s (motor: 6010-8) -->
+    <limit lower="-0.7853981634" upper="0.7853981634" effort="11.0" velocity="12.5663706144"/>
+    <!-- friction: no-load current 0.4A x torque constant 0.47N·m/A = 0.188N·m (Coulomb friction estimate); damping: not given in datasheet, kept at 0.0 -->
+    <dynamics damping="0.0" friction="0.188"/>
   </joint>
   <link name="back_right_upper_leg_link">
@@ -459,6 +479,8 @@
     <child link="back_right_upper_leg_link"/>
     <axis xyz="0 1 0"/>
-    <limit lower="-1.57079632679" upper="2.59" effort="40.0" velocity="4.0"/>
-    <dynamics damping="0.0" friction="0.0"/>
+    <!-- upper joint limit: -90~140 deg | effort: stall torque 11N·m, velocity: rated speed 120rpm = 12.5663706144 rad/s (motor: 6010-8) -->
+    <limit lower="-1.5707963268" upper="2.4434609528" effort="11.0" velocity="12.5663706144"/>
+    <!-- friction: no-load current 0.4A x torque constant 0.47N·m/A = 0.188N·m (Coulomb friction estimate); damping: not given in datasheet, kept at 0.0 -->
+    <dynamics damping="0.0" friction="0.188"/>
   </joint>
   <link name="back_right_lower_leg_link">
@@ -482,6 +504,8 @@
     <child link="back_right_lower_leg_link"/>
     <axis xyz="0 1 0"/>
-    <limit lower="-2.4783675378" upper="2.4783675378" effort="40.0" velocity="4.0"/>
-    <dynamics damping="0.0" friction="0.0"/>
+    <!-- lower joint limit: -135~135 deg | effort: stall torque 11N·m, velocity: rated speed 120rpm = 12.5663706144 rad/s (motor: 6010-8) -->
+    <limit lower="-2.3561944902" upper="2.3561944902" effort="11.0" velocity="12.5663706144"/>
+    <!-- friction: no-load current 0.4A x torque constant 0.47N·m/A = 0.188N·m (Coulomb friction estimate); damping: not given in datasheet, kept at 0.0 -->
+    <dynamics damping="0.0" friction="0.188"/>
   </joint>
   <link name="back_right_foot_link">
