Commit message: calibration 구현

File: src/quattro_description/urdf/quattro.urdf.xacro (robot description, xacro)
@@ -1,4 +1,10 @@
 <?xml version="1.0"?>
 <robot xmlns:xacro="http://www.ros.org/wiki/xacro" name="quattro">
+  <xacro:arg
+    name="calibration_file"
+    default="../config/calibration.yaml"/>
+  <xacro:property
+    name="hardware_calibration"
+    value="${xacro.load_yaml('$(arg calibration_file)')['joints']}"/>
   <!--
     Mesh directory:
@@ -35,4 +41,21 @@
     </collision>
   </xacro:macro>
+  <xacro:macro name="quattro_hardware_joint" params="name lower upper">
+    <joint name="${name}">
+      <command_interface name="position">
+        <param name="min">${lower}</param>
+        <param name="max">${upper}</param>
+      </command_interface>
+      <state_interface name="position"/>
+      <state_interface name="velocity"/>
+      <state_interface name="effort"/>
+      <param name="can_interface">${hardware_calibration[name]['can_interface']}</param>
+      <param name="can_id">${hardware_calibration[name]['can_id']}</param>
+      <param name="direction">${hardware_calibration[name]['direction']}</param>
+      <param name="offset">${hardware_calibration[name]['offset']}</param>
+      <param name="kp">${hardware_calibration[name]['kp']}</param>
+      <param name="kd">${hardware_calibration[name]['kd']}</param>
+    </joint>
+  </xacro:macro>
   <!-- ================================================================ -->
   <!-- Base                                                             -->
@@ -412,3 +435,25 @@
     <child link="back_right_foot_link"/>
   </joint>
+  <ros2_control name="QuattroSystem" type="system">
+    <hardware>
+      <plugin>quattro_hardware/QuattroSystem</plugin>
+      <param name="feedback_timeout_ms">100</param>
+      <param name="startup_timeout_ms">1000</param>
+      <param name="command_timeout_ms">100</param>
+      <param name="motor_velocity_limit">50.0</param>
+      <param name="motor_current_limit">20.0</param>
+    </hardware>
+    <xacro:quattro_hardware_joint name="front_left_hip_joint" lower="-1.04" upper="1.04"/>
+    <xacro:quattro_hardware_joint name="front_left_upper_leg_joint" lower="-1.57079632679" upper="2.59"/>
+    <xacro:quattro_hardware_joint name="front_left_lower_leg_joint" lower="-2.9" upper="1.57079632679"/>
+    <xacro:quattro_hardware_joint name="front_right_hip_joint" lower="-1.04" upper="1.04"/>
+    <xacro:quattro_hardware_joint name="front_right_upper_leg_joint" lower="-1.57079632679" upper="2.59"/>
+    <xacro:quattro_hardware_joint name="front_right_lower_leg_joint" lower="-2.9" upper="1.57079632679"/>
+    <xacro:quattro_hardware_joint name="back_left_hip_joint" lower="-1.04" upper="1.04"/>
+    <xacro:quattro_hardware_joint name="back_left_upper_leg_joint" lower="-1.57079632679" upper="2.59"/>
+    <xacro:quattro_hardware_joint name="back_left_lower_leg_joint" lower="-2.9" upper="1.57079632679"/>
+    <xacro:quattro_hardware_joint name="back_right_hip_joint" lower="-1.04" upper="1.04"/>
+    <xacro:quattro_hardware_joint name="back_right_upper_leg_joint" lower="-1.57079632679" upper="2.59"/>
+    <xacro:quattro_hardware_joint name="back_right_lower_leg_joint" lower="-2.9" upper="1.57079632679"/>
+  </ros2_control>
 </robot>

Commit message: Gazebo 구현

File: src/quattro_description/urdf/quattro.urdf.xacro (robot description, xacro)
@@ -4,4 +4,8 @@
     name="calibration_file"
     default="../config/calibration.yaml"/>
+  <xacro:arg name="simulation" default="false"/>
+  <xacro:arg
+    name="simulation_controllers"
+    default="../../quattro_gazebo/config/gazebo_controllers.yaml"/>
   <xacro:property
     name="hardware_calibration"
@@ -58,4 +62,17 @@
     </joint>
   </xacro:macro>
+  <xacro:macro name="quattro_simulation_joint" params="name lower upper initial_value">
+    <joint name="${name}">
+      <command_interface name="position">
+        <param name="min">${lower}</param>
+        <param name="max">${upper}</param>
+      </command_interface>
+      <state_interface name="position">
+        <param name="initial_value">${initial_value}</param>
+      </state_interface>
+      <state_interface name="velocity"/>
+      <state_interface name="effort"/>
+    </joint>
+  </xacro:macro>
   <!-- ================================================================ -->
   <!-- Base                                                             -->
@@ -435,25 +452,53 @@
     <child link="back_right_foot_link"/>
   </joint>
-  <ros2_control name="QuattroSystem" type="system">
-    <hardware>
-      <plugin>quattro_hardware/QuattroSystem</plugin>
-      <param name="feedback_timeout_ms">100</param>
-      <param name="startup_timeout_ms">1000</param>
-      <param name="command_timeout_ms">100</param>
-      <param name="motor_velocity_limit">50.0</param>
-      <param name="motor_current_limit">20.0</param>
-    </hardware>
-    <xacro:quattro_hardware_joint name="front_left_hip_joint" lower="-1.04" upper="1.04"/>
-    <xacro:quattro_hardware_joint name="front_left_upper_leg_joint" lower="-1.57079632679" upper="2.59"/>
-    <xacro:quattro_hardware_joint name="front_left_lower_leg_joint" lower="-2.9" upper="1.57079632679"/>
-    <xacro:quattro_hardware_joint name="front_right_hip_joint" lower="-1.04" upper="1.04"/>
-    <xacro:quattro_hardware_joint name="front_right_upper_leg_joint" lower="-1.57079632679" upper="2.59"/>
-    <xacro:quattro_hardware_joint name="front_right_lower_leg_joint" lower="-2.9" upper="1.57079632679"/>
-    <xacro:quattro_hardware_joint name="back_left_hip_joint" lower="-1.04" upper="1.04"/>
-    <xacro:quattro_hardware_joint name="back_left_upper_leg_joint" lower="-1.57079632679" upper="2.59"/>
-    <xacro:quattro_hardware_joint name="back_left_lower_leg_joint" lower="-2.9" upper="1.57079632679"/>
-    <xacro:quattro_hardware_joint name="back_right_hip_joint" lower="-1.04" upper="1.04"/>
-    <xacro:quattro_hardware_joint name="back_right_upper_leg_joint" lower="-1.57079632679" upper="2.59"/>
-    <xacro:quattro_hardware_joint name="back_right_lower_leg_joint" lower="-2.9" upper="1.57079632679"/>
-  </ros2_control>
+  <xacro:unless value="$(arg simulation)">
+    <ros2_control name="QuattroSystem" type="system">
+      <hardware>
+        <plugin>quattro_hardware/QuattroSystem</plugin>
+        <param name="feedback_timeout_ms">100</param>
+        <param name="startup_timeout_ms">1000</param>
+        <param name="command_timeout_ms">100</param>
+        <param name="motor_velocity_limit">50.0</param>
+        <param name="motor_current_limit">20.0</param>
+      </hardware>
+      <xacro:quattro_hardware_joint name="front_left_hip_joint" lower="-1.04" upper="1.04"/>
+      <xacro:quattro_hardware_joint name="front_left_upper_leg_joint" lower="-1.57079632679" upper="2.59"/>
+      <xacro:quattro_hardware_joint name="front_left_lower_leg_joint" lower="-2.9" upper="1.57079632679"/>
+      <xacro:quattro_hardware_joint name="front_right_hip_joint" lower="-1.04" upper="1.04"/>
+      <xacro:quattro_hardware_joint name="front_right_upper_leg_joint" lower="-1.57079632679" upper="2.59"/>
+      <xacro:quattro_hardware_joint name="front_right_lower_leg_joint" lower="-2.9" upper="1.57079632679"/>
+      <xacro:quattro_hardware_joint name="back_left_hip_joint" lower="-1.04" upper="1.04"/>
+      <xacro:quattro_hardware_joint name="back_left_upper_leg_joint" lower="-1.57079632679" upper="2.59"/>
+      <xacro:quattro_hardware_joint name="back_left_lower_leg_joint" lower="-2.9" upper="1.57079632679"/>
+      <xacro:quattro_hardware_joint name="back_right_hip_joint" lower="-1.04" upper="1.04"/>
+      <xacro:quattro_hardware_joint name="back_right_upper_leg_joint" lower="-1.57079632679" upper="2.59"/>
+      <xacro:quattro_hardware_joint name="back_right_lower_leg_joint" lower="-2.9" upper="1.57079632679"/>
+    </ros2_control>
+  </xacro:unless>
+  <xacro:if value="$(arg simulation)">
+    <ros2_control name="GazeboSimSystem" type="system">
+      <hardware>
+        <plugin>gz_ros2_control/GazeboSimSystem</plugin>
+      </hardware>
+      <xacro:quattro_simulation_joint name="front_left_hip_joint" lower="-1.04" upper="1.04" initial_value="0.0"/>
+      <xacro:quattro_simulation_joint name="front_left_upper_leg_joint" lower="-1.57079632679" upper="2.59" initial_value="0.63356747785"/>
+      <xacro:quattro_simulation_joint name="front_left_lower_leg_joint" lower="-2.9" upper="1.57079632679" initial_value="-1.53223802029"/>
+      <xacro:quattro_simulation_joint name="front_right_hip_joint" lower="-1.04" upper="1.04" initial_value="0.0"/>
+      <xacro:quattro_simulation_joint name="front_right_upper_leg_joint" lower="-1.57079632679" upper="2.59" initial_value="0.63356747785"/>
+      <xacro:quattro_simulation_joint name="front_right_lower_leg_joint" lower="-2.9" upper="1.57079632679" initial_value="-1.53223802029"/>
+      <xacro:quattro_simulation_joint name="back_left_hip_joint" lower="-1.04" upper="1.04" initial_value="0.0"/>
+      <xacro:quattro_simulation_joint name="back_left_upper_leg_joint" lower="-1.57079632679" upper="2.59" initial_value="0.63356747785"/>
+      <xacro:quattro_simulation_joint name="back_left_lower_leg_joint" lower="-2.9" upper="1.57079632679" initial_value="-1.53223802029"/>
+      <xacro:quattro_simulation_joint name="back_right_hip_joint" lower="-1.04" upper="1.04" initial_value="0.0"/>
+      <xacro:quattro_simulation_joint name="back_right_upper_leg_joint" lower="-1.57079632679" upper="2.59" initial_value="0.63356747785"/>
+      <xacro:quattro_simulation_joint name="back_right_lower_leg_joint" lower="-2.9" upper="1.57079632679" initial_value="-1.53223802029"/>
+    </ros2_control>
+    <gazebo>
+      <plugin
+        filename="libgz_ros2_control-system.so"
+        name="gz_ros2_control::GazeboSimROS2ControlPlugin">
+        <parameters>$(arg simulation_controllers)</parameters>
+      </plugin>
+    </gazebo>
+  </xacro:if>
 </robot>

Commit message: gim6010_driver 수정

File: src/quattro_description/urdf/quattro.urdf.xacro (robot description, xacro)
@@ -5,4 +5,9 @@
     default="../config/calibration.yaml"/>
   <xacro:arg name="simulation" default="false"/>
+  <xacro:arg name="hardware_control_method" default="direct_position"/>
+  <xacro:arg name="apply_position_gains" default="false"/>
+  <xacro:arg name="position_gain" default="0.0"/>
+  <xacro:arg name="velocity_gain" default="0.0"/>
+  <xacro:arg name="velocity_integrator_gain" default="0.0"/>
   <xacro:arg
     name="simulation_controllers"
@@ -11,4 +16,5 @@
     name="hardware_calibration"
     value="${xacro.load_yaml('$(arg calibration_file)')['joints']}"/>
+  <xacro:property name="hardware_control_method" value="$(arg hardware_control_method)"/>
   <!--
     Mesh directory:
@@ -47,8 +53,29 @@
   <xacro:macro name="quattro_hardware_joint" params="name lower upper">
     <joint name="${name}">
-      <command_interface name="position">
-        <param name="min">${lower}</param>
-        <param name="max">${upper}</param>
-      </command_interface>
+      <xacro:if value="${hardware_control_method == 'direct_position'}">
+        <command_interface name="position">
+          <param name="min">${lower}</param>
+          <param name="max">${upper}</param>
+        </command_interface>
+      </xacro:if>
+      <xacro:if value="${hardware_control_method == 'mit'}">
+        <command_interface name="position"><param name="min">${lower}</param><param name="max">${upper}</param></command_interface>
+        <command_interface name="velocity"><param name="min">-4.0</param><param name="max">4.0</param></command_interface>
+        <command_interface name="kp"><param name="min">0.0</param><param name="max">500.0</param></command_interface>
+        <command_interface name="kd"><param name="min">0.0</param><param name="max">5.0</param></command_interface>
+        <command_interface name="effort"><param name="min">-10.0</param><param name="max">10.0</param></command_interface>
+      </xacro:if>
+      <xacro:if value="${hardware_control_method == 'direct_velocity'}">
+        <command_interface name="velocity">
+          <param name="min">-4.0</param>
+          <param name="max">4.0</param>
+        </command_interface>
+      </xacro:if>
+      <xacro:if value="${hardware_control_method == 'direct_torque'}">
+        <command_interface name="effort">
+          <param name="min">-10.0</param>
+          <param name="max">10.0</param>
+        </command_interface>
+      </xacro:if>
       <state_interface name="position"/>
       <state_interface name="velocity"/>
@@ -58,6 +85,7 @@
       <param name="direction">${hardware_calibration[name]['direction']}</param>
       <param name="offset">${hardware_calibration[name]['offset']}</param>
-      <param name="kp">${hardware_calibration[name]['kp']}</param>
-      <param name="kd">${hardware_calibration[name]['kd']}</param>
+      <param name="gear_ratio">8.0</param>
+      <param name="mit_kp">${hardware_calibration[name]['kp']}</param>
+      <param name="mit_kd">${hardware_calibration[name]['kd']}</param>
     </joint>
   </xacro:macro>
@@ -456,10 +484,16 @@
       <hardware>
         <plugin>quattro_hardware/QuattroSystem</plugin>
-        <param name="feedback_timeout_ms">100</param>
-        <param name="heartbeat_timeout_ms">300</param>
+        <param name="control_method">${hardware_control_method}</param>
+        <param name="apply_position_gains">$(arg apply_position_gains)</param>
+        <param name="position_gain">$(arg position_gain)</param>
+        <param name="velocity_gain">$(arg velocity_gain)</param>
+        <param name="velocity_integrator_gain">$(arg velocity_integrator_gain)</param>
+        <param name="feedback_timeout_ms">150</param>
+        <param name="heartbeat_timeout_ms">400</param>
         <param name="startup_timeout_ms">1000</param>
-        <param name="command_timeout_ms">100</param>
-        <param name="motor_velocity_limit">50.0</param>
-        <param name="motor_current_limit">20.0</param>
+        <param name="command_timeout_ms">250</param>
+        <param name="scheduling_warning_ms">50</param>
+        <param name="rotor_velocity_limit_rev_s">5.0</param>
+        <param name="motor_current_limit_a">5.0</param>
         <param name="engagement_duration_ms">1000</param>
         <param name="telemetry_period_ms">500</param>

Commit message: Direct Position Control 구현

File: src/quattro_description/urdf/quattro.urdf.xacro (robot description, xacro)
@@ -5,5 +5,4 @@
     default="../config/calibration.yaml"/>
   <xacro:arg name="simulation" default="false"/>
-  <xacro:arg name="hardware_control_method" default="mit"/>
   <xacro:arg name="apply_position_gains" default="false"/>
   <xacro:arg name="position_gain" default="0.0"/>
@@ -17,5 +16,4 @@
     name="hardware_calibration"
     value="${xacro.load_yaml('$(arg calibration_file)')['joints']}"/>
-  <xacro:property name="hardware_control_method" value="$(arg hardware_control_method)"/>
   <!--
     Mesh directory:
@@ -54,29 +52,8 @@
   <xacro:macro name="quattro_hardware_joint" params="name lower upper">
     <joint name="${name}">
-      <xacro:if value="${hardware_control_method == 'direct_position'}">
-        <command_interface name="position">
-          <param name="min">${lower}</param>
-          <param name="max">${upper}</param>
-        </command_interface>
-      </xacro:if>
-      <xacro:if value="${hardware_control_method == 'mit'}">
-        <command_interface name="position"><param name="min">${lower}</param><param name="max">${upper}</param></command_interface>
-        <command_interface name="velocity"><param name="min">-4.0</param><param name="max">4.0</param></command_interface>
-        <command_interface name="kp"/>
-        <command_interface name="kd"/>
-        <command_interface name="effort"><param name="min">-10.0</param><param name="max">10.0</param></command_interface>
-      </xacro:if>
-      <xacro:if value="${hardware_control_method == 'direct_velocity'}">
-        <command_interface name="velocity">
-          <param name="min">-4.0</param>
-          <param name="max">4.0</param>
-        </command_interface>
-      </xacro:if>
-      <xacro:if value="${hardware_control_method == 'direct_torque'}">
-        <command_interface name="effort">
-          <param name="min">-10.0</param>
-          <param name="max">10.0</param>
-        </command_interface>
-      </xacro:if>
+      <command_interface name="position">
+        <param name="min">${lower}</param>
+        <param name="max">${upper}</param>
+      </command_interface>
       <state_interface name="position"/>
       <state_interface name="velocity"/>
@@ -88,35 +65,12 @@
       <param name="gear_ratio">8.0</param>
       <param name="current_limit">${hardware_calibration[name].get('current_limit', 5.0)}</param>
-      <param name="mit_kp">${hardware_calibration[name]['kp']}</param>
-      <param name="mit_kd">${hardware_calibration[name]['kd']}</param>
     </joint>
   </xacro:macro>
-  <!--
-    simulation:=true always uses gz_ros2_control/GazeboSimSystem, whose
-    stock implementation only understands the standard interface names
-    (position/velocity/effort); it has no notion of the GIM6010 MIT
-    frame's per-joint kp/kd fields. So unlike the real-hardware branch
-    above, this macro cannot expose position/velocity/kp/kd/effort for
-    hardware_control_method=mit. Instead it exposes a single `effort`
-    command interface, and quattro_controllers/MitTrajectoryController's
-    command_mode=effort_emulation computes the MIT PD law on the host and
-    writes the result there (docs/packages/quattro_controllers.md,
-    docs/gazebo.md). Every other hardware_control_method keeps the
-    original position-only interface, unchanged.
-  -->
   <xacro:macro name="quattro_simulation_joint" params="name lower upper initial_value">
     <joint name="${name}">
-      <xacro:if value="${hardware_control_method == 'mit'}">
-        <command_interface name="effort">
-          <param name="min">-40.0</param>
-          <param name="max">40.0</param>
-        </command_interface>
-      </xacro:if>
-      <xacro:unless value="${hardware_control_method == 'mit'}">
-        <command_interface name="position">
-          <param name="min">${lower}</param>
-          <param name="max">${upper}</param>
-        </command_interface>
-      </xacro:unless>
+      <command_interface name="position">
+        <param name="min">${lower}</param>
+        <param name="max">${upper}</param>
+      </command_interface>
       <state_interface name="position">
         <param name="initial_value">${initial_value}</param>
@@ -507,5 +461,4 @@
       <hardware>
         <plugin>quattro_hardware/QuattroSystem</plugin>
-        <param name="control_method">${hardware_control_method}</param>
         <param name="apply_position_gains">$(arg apply_position_gains)</param>
         <param name="position_gain">$(arg position_gain)</param>
@@ -521,5 +474,4 @@
         <param name="rotor_velocity_limit_rev_s">5.0</param>
         <param name="motor_current_limit_a">5.0</param>
-        <param name="engagement_duration_ms">1000</param>
         <param name="telemetry_period_ms">500</param>
       </hardware>
