Commit message: URDF 수정

File: src/quattro_description/urdf/quattro.urdf.xacro (robot description, xacro)
@@ -19,5 +19,5 @@
     Mesh directory:
       package://quattro_description/meshes/stl/
-    The same STL is used for both visual and collision geometry.
+    STL files are used for visual geometry only. Collision geometry uses primitives.
     The original URDF used scale="1 1 1", so that value is preserved.
     Change mesh_scale to "0.001 0.001 0.001" only when the STL is exported in millimetres.
@@ -34,6 +34,5 @@
     <color rgba="0.6 0.6 0.6 1.0"/>
   </material>
-  <!-- Creates visual and collision elements from the same STL file. -->
-  <xacro:macro name="stl_visual_collision" params="filename material_name">
+  <xacro:macro name="stl_visual" params="filename material_name">
     <visual>
       <origin xyz="0 0 0" rpy="0 0 0"/>
@@ -43,8 +42,26 @@
       <material name="${material_name}"/>
     </visual>
-    <collision>
-      <origin xyz="0 0 0" rpy="0 0 0"/>
+  </xacro:macro>
+  <xacro:macro name="box_collision" params="xyz rpy size">
+    <collision>
+      <origin xyz="${xyz}" rpy="${rpy}"/>
       <geometry>
-        <mesh filename="${mesh_prefix}/${filename}" scale="${mesh_scale}"/>
+        <box size="${size}"/>
+      </geometry>
+    </collision>
+  </xacro:macro>
+  <xacro:macro name="cylinder_collision" params="xyz rpy radius length">
+    <collision>
+      <origin xyz="${xyz}" rpy="${rpy}"/>
+      <geometry>
+        <cylinder radius="${radius}" length="${length}"/>
+      </geometry>
+    </collision>
+  </xacro:macro>
+  <xacro:macro name="sphere_collision" params="xyz radius">
+    <collision>
+      <origin xyz="${xyz}" rpy="0 0 0"/>
+      <geometry>
+        <sphere radius="${radius}"/>
       </geometry>
     </collision>
@@ -84,5 +101,6 @@
   <!-- ================================================================ -->
   <link name="base_link">
-    <xacro:stl_visual_collision filename="body_frame.stl" material_name="orange"/>
+    <xacro:stl_visual filename="body_frame.stl" material_name="orange"/>
+    <xacro:box_collision xyz="0 0 0" rpy="0 0 0" size="0.43 0.14 0.10"/>
     <inertial>
       <origin xyz="0.001210 -0.000887 -0.007933" rpy="0 0 0"/>
@@ -101,5 +119,6 @@
   <!-- ================================================================ -->
   <link name="front_left_hip_link">
-    <xacro:stl_visual_collision filename="front_left_hip.stl" material_name="black"/>
+    <xacro:stl_visual filename="front_left_hip.stl" material_name="black"/>
+    <xacro:cylinder_collision xyz="0 0.04525 0" rpy="1.57079632679 0 0" radius="0.035" length="0.075"/>
     <inertial>
       <origin xyz="-0.003 -0.000913 -0.000423" rpy="0 0 0"/>
@@ -123,5 +142,6 @@
   </joint>
   <link name="front_left_upper_leg_link">
-    <xacro:stl_visual_collision filename="left_upper_leg.stl" material_name="black"/>
+    <xacro:stl_visual filename="left_upper_leg.stl" material_name="black"/>
+    <xacro:box_collision xyz="0 0 -0.105" rpy="0 0 0" size="0.045 0.045 0.18"/>
     <inertial>
       <origin xyz="0.00011 -0.017289 -0.042003" rpy="0 0 0"/>
@@ -145,5 +165,6 @@
   </joint>
   <link name="front_left_lower_leg_link">
-    <xacro:stl_visual_collision filename="left_lower_leg.stl" material_name="black"/>
+    <xacro:stl_visual filename="left_lower_leg.stl" material_name="black"/>
+    <xacro:cylinder_collision xyz="0 0 -0.105" rpy="0 0 0" radius="0.018" length="0.18"/>
     <inertial>
       <origin xyz="-0.000176 0 -0.034133" rpy="0 0 0"/>
@@ -163,5 +184,5 @@
     <child link="front_left_lower_leg_link"/>
     <axis xyz="0 1 0"/>
-    <limit lower="-2.9" upper="1.57079632679" effort="40.0" velocity="4.0"/>
+    <limit lower="-2.4783675378" upper="2.4783675378" effort="40.0" velocity="4.0"/>
     <dynamics damping="0.0" friction="0.0"/>
   </joint>
@@ -191,5 +212,6 @@
   <!-- ================================================================ -->
   <link name="front_right_hip_link">
-    <xacro:stl_visual_collision filename="front_right_hip.stl" material_name="black"/>
+    <xacro:stl_visual filename="front_right_hip.stl" material_name="black"/>
+    <xacro:cylinder_collision xyz="0 -0.04525 0" rpy="1.57079632679 0 0" radius="0.035" length="0.075"/>
     <inertial>
       <origin xyz="-0.003304 0.000913 -0.000118" rpy="0 0 0"/>
@@ -213,5 +235,6 @@
   </joint>
   <link name="front_right_upper_leg_link">
-    <xacro:stl_visual_collision filename="right_upper_leg.stl" material_name="black"/>
+    <xacro:stl_visual filename="right_upper_leg.stl" material_name="black"/>
+    <xacro:box_collision xyz="0 0 -0.105" rpy="0 0 0" size="0.045 0.045 0.18"/>
     <inertial>
       <origin xyz="-0.00011 0.017289 -0.042003" rpy="0 0 0"/>
@@ -235,5 +258,6 @@
   </joint>
   <link name="front_right_lower_leg_link">
-    <xacro:stl_visual_collision filename="right_lower_leg.stl" material_name="black"/>
+    <xacro:stl_visual filename="right_lower_leg.stl" material_name="black"/>
+    <xacro:cylinder_collision xyz="0 0 -0.105" rpy="0 0 0" radius="0.018" length="0.18"/>
     <inertial>
       <origin xyz="0.000176 0 -0.034133" rpy="0 0 0"/>
@@ -253,5 +277,5 @@
     <child link="front_right_lower_leg_link"/>
     <axis xyz="0 1 0"/>
-    <limit lower="-2.9" upper="1.57079632679" effort="40.0" velocity="4.0"/>
+    <limit lower="-2.4783675378" upper="2.4783675378" effort="40.0" velocity="4.0"/>
     <dynamics damping="0.0" friction="0.0"/>
   </joint>
@@ -281,5 +305,6 @@
   <!-- ================================================================ -->
   <link name="back_left_hip_link">
-    <xacro:stl_visual_collision filename="back_left_hip.stl" material_name="black"/>
+    <xacro:stl_visual filename="back_left_hip.stl" material_name="black"/>
+    <xacro:cylinder_collision xyz="0 0.04525 0" rpy="1.57079632679 0 0" radius="0.035" length="0.075"/>
     <inertial>
       <origin xyz="0.003304 -0.000713 -0.000118" rpy="0 0 0"/>
@@ -303,5 +328,6 @@
   </joint>
   <link name="back_left_upper_leg_link">
-    <xacro:stl_visual_collision filename="left_upper_leg.stl" material_name="black"/>
+    <xacro:stl_visual filename="left_upper_leg.stl" material_name="black"/>
+    <xacro:box_collision xyz="0 0 -0.105" rpy="0 0 0" size="0.045 0.045 0.18"/>
     <inertial>
       <origin xyz="0.00011 -0.017289 -0.042003" rpy="0 0 0"/>
@@ -325,5 +351,6 @@
   </joint>
   <link name="back_left_lower_leg_link">
-    <xacro:stl_visual_collision filename="left_lower_leg.stl" material_name="black"/>
+    <xacro:stl_visual filename="left_lower_leg.stl" material_name="black"/>
+    <xacro:cylinder_collision xyz="0 0 -0.105" rpy="0 0 0" radius="0.018" length="0.18"/>
     <inertial>
       <origin xyz="-0.000176 0 -0.034133" rpy="0 0 0"/>
@@ -343,5 +370,5 @@
     <child link="back_left_lower_leg_link"/>
     <axis xyz="0 1 0"/>
-    <limit lower="-2.9" upper="1.57079632679" effort="40.0" velocity="4.0"/>
+    <limit lower="-2.4783675378" upper="2.4783675378" effort="40.0" velocity="4.0"/>
     <dynamics damping="0.0" friction="0.0"/>
   </joint>
@@ -371,5 +398,6 @@
   <!-- ================================================================ -->
   <link name="back_right_hip_link">
-    <xacro:stl_visual_collision filename="back_right_hip.stl" material_name="black"/>
+    <xacro:stl_visual filename="back_right_hip.stl" material_name="black"/>
+    <xacro:cylinder_collision xyz="0 -0.04525 0" rpy="1.57079632679 0 0" radius="0.035" length="0.075"/>
     <inertial>
       <origin xyz="0.003 0.001113 -0.000423" rpy="0 0 0"/>
@@ -393,5 +421,6 @@
   </joint>
   <link name="back_right_upper_leg_link">
-    <xacro:stl_visual_collision filename="right_upper_leg.stl" material_name="black"/>
+    <xacro:stl_visual filename="right_upper_leg.stl" material_name="black"/>
+    <xacro:box_collision xyz="0 0 -0.105" rpy="0 0 0" size="0.045 0.045 0.18"/>
     <inertial>
       <origin xyz="-0.00011 0.017289 -0.042003" rpy="0 0 0"/>
@@ -415,5 +444,6 @@
   </joint>
   <link name="back_right_lower_leg_link">
-    <xacro:stl_visual_collision filename="right_lower_leg.stl" material_name="black"/>
+    <xacro:stl_visual filename="right_lower_leg.stl" material_name="black"/>
+    <xacro:cylinder_collision xyz="0 0 -0.105" rpy="0 0 0" radius="0.018" length="0.18"/>
     <inertial>
       <origin xyz="0.000176 0 -0.034133" rpy="0 0 0"/>
@@ -433,5 +463,5 @@
     <child link="back_right_lower_leg_link"/>
     <axis xyz="0 1 0"/>
-    <limit lower="-2.9" upper="1.57079632679" effort="40.0" velocity="4.0"/>
+    <limit lower="-2.4783675378" upper="2.4783675378" effort="40.0" velocity="4.0"/>
     <dynamics damping="0.0" friction="0.0"/>
   </joint>

Commit message: RViz2 시각화 수정

File: src/quattro_description/urdf/quattro.urdf.xacro (robot description, xacro)
@@ -10,4 +10,6 @@
   <xacro:arg name="velocity_integrator_gain" default="0.0"/>
   <xacro:arg name="motor_activation_interval_ms" default="100"/>
+  <xacro:arg name="visual_color_override" default="false"/>
+  <xacro:arg name="visual_color" default="0.1 0.1 0.1 1.0"/>
   <xacro:arg
     name="simulation_controllers"
@@ -34,4 +36,7 @@
     <color rgba="0.6 0.6 0.6 1.0"/>
   </material>
+  <material name="visual_color_override">
+    <color rgba="$(arg visual_color)"/>
+  </material>
   <xacro:macro name="stl_visual" params="filename material_name">
     <visual>
@@ -40,5 +45,10 @@
         <mesh filename="${mesh_prefix}/${filename}" scale="${mesh_scale}"/>
       </geometry>
-      <material name="${material_name}"/>
+      <xacro:if value="$(arg visual_color_override)">
+        <material name="visual_color_override"/>
+      </xacro:if>
+      <xacro:unless value="$(arg visual_color_override)">
+        <material name="${material_name}"/>
+      </xacro:unless>
     </visual>
   </xacro:macro>
@@ -191,5 +201,10 @@
       <origin xyz="0 0 0" rpy="0 0 0"/>
       <geometry><sphere radius="0.025"/></geometry>
-      <material name="grey"/>
+      <xacro:if value="$(arg visual_color_override)">
+        <material name="visual_color_override"/>
+      </xacro:if>
+      <xacro:unless value="$(arg visual_color_override)">
+        <material name="grey"/>
+      </xacro:unless>
     </visual>
     <collision>
@@ -284,5 +299,10 @@
       <origin xyz="0 0 0" rpy="0 0 0"/>
       <geometry><sphere radius="0.025"/></geometry>
-      <material name="grey"/>
+      <xacro:if value="$(arg visual_color_override)">
+        <material name="visual_color_override"/>
+      </xacro:if>
+      <xacro:unless value="$(arg visual_color_override)">
+        <material name="grey"/>
+      </xacro:unless>
     </visual>
     <collision>
@@ -377,5 +397,10 @@
       <origin xyz="0 0 0" rpy="0 0 0"/>
       <geometry><sphere radius="0.025"/></geometry>
-      <material name="grey"/>
+      <xacro:if value="$(arg visual_color_override)">
+        <material name="visual_color_override"/>
+      </xacro:if>
+      <xacro:unless value="$(arg visual_color_override)">
+        <material name="grey"/>
+      </xacro:unless>
     </visual>
     <collision>
@@ -470,5 +495,10 @@
       <origin xyz="0 0 0" rpy="0 0 0"/>
       <geometry><sphere radius="0.025"/></geometry>
-      <material name="grey"/>
+      <xacro:if value="$(arg visual_color_override)">
+        <material name="visual_color_override"/>
+      </xacro:if>
+      <xacro:unless value="$(arg visual_color_override)">
+        <material name="grey"/>
+      </xacro:unless>
     </visual>
     <collision>

Commit message: 캘리브레이션 Direct Position 으로 변경

File: src/quattro_description/urdf/quattro.urdf.xacro (robot description, xacro)
@@ -5,8 +5,4 @@
     default="../config/calibration.yaml"/>
   <xacro:arg name="simulation" default="false"/>
-  <xacro:arg name="apply_position_gains" default="false"/>
-  <xacro:arg name="position_gain" default="0.0"/>
-  <xacro:arg name="velocity_gain" default="0.0"/>
-  <xacro:arg name="velocity_integrator_gain" default="0.0"/>
   <xacro:arg name="motor_activation_interval_ms" default="100"/>
   <xacro:arg name="visual_color_override" default="false"/>
@@ -15,7 +11,7 @@
     name="simulation_controllers"
     default="../../quattro_gazebo/config/gazebo_controllers.yaml"/>
-  <xacro:property
-    name="hardware_calibration"
-    value="${xacro.load_yaml('$(arg calibration_file)')['joints']}"/>
+  <xacro:property name="calibration" value="${xacro.load_yaml('$(arg calibration_file)')}"/>
+  <xacro:property name="hardware_calibration" value="${calibration['joints']}"/>
+  <xacro:property name="direct_position" value="${calibration['direct_position']}"/>
   <!--
     Mesh directory:
@@ -91,5 +87,4 @@
       <param name="offset">${hardware_calibration[name]['offset']}</param>
       <param name="gear_ratio">8.0</param>
-      <param name="current_limit">${hardware_calibration[name].get('current_limit', 5.0)}</param>
     </joint>
   </xacro:macro>
@@ -521,8 +516,8 @@
       <hardware>
         <plugin>quattro_hardware/QuattroSystem</plugin>
-        <param name="apply_position_gains">$(arg apply_position_gains)</param>
-        <param name="position_gain">$(arg position_gain)</param>
-        <param name="velocity_gain">$(arg velocity_gain)</param>
-        <param name="velocity_integrator_gain">$(arg velocity_integrator_gain)</param>
+        <param name="current_limit">${direct_position['current_limit']}</param>
+        <param name="position_gain">${direct_position['position_gain']}</param>
+        <param name="velocity_gain">${direct_position['velocity_gain']}</param>
+        <param name="velocity_integrator_gain">${direct_position['velocity_integrator_gain']}</param>
         <param name="feedback_timeout_ms">150</param>
         <param name="feedback_request_period_ms">50</param>
@@ -533,5 +528,4 @@
         <param name="scheduling_warning_ms">50</param>
         <param name="rotor_velocity_limit_rev_s">5.0</param>
-        <param name="motor_current_limit_a">5.0</param>
         <param name="telemetry_period_ms">500</param>
       </hardware>

Commit message: 실기 검증 및 PID 튜닝

File: src/quattro_description/urdf/quattro.urdf.xacro (robot description, xacro)
@@ -5,5 +5,4 @@
     default="../config/calibration.yaml"/>
   <xacro:arg name="simulation" default="false"/>
-  <xacro:arg name="motor_activation_interval_ms" default="100"/>
   <xacro:arg name="visual_color_override" default="false"/>
   <xacro:arg name="visual_color" default="0.1 0.1 0.1 1.0"/>
@@ -13,5 +12,5 @@
   <xacro:property name="calibration" value="${xacro.load_yaml('$(arg calibration_file)')}"/>
   <xacro:property name="hardware_calibration" value="${calibration['joints']}"/>
-  <xacro:property name="direct_position" value="${calibration['direct_position']}"/>
+  <xacro:property name="position_control" value="${calibration['position_control']}"/>
   <!--
     Mesh directory:
@@ -516,12 +515,32 @@
       <hardware>
         <plugin>quattro_hardware/QuattroSystem</plugin>
-        <param name="current_limit">${direct_position['current_limit']}</param>
-        <param name="position_gain">${direct_position['position_gain']}</param>
-        <param name="velocity_gain">${direct_position['velocity_gain']}</param>
-        <param name="velocity_integrator_gain">${direct_position['velocity_integrator_gain']}</param>
+        <param name="current_limit">${position_control['current_limit']}</param>
+        <param name="position_gain">${position_control['position_gain']}</param>
+        <param name="velocity_gain">${position_control['velocity_gain']}</param>
+        <param name="velocity_integrator_gain">${position_control['velocity_integrator_gain']}</param>
         <param name="feedback_timeout_ms">150</param>
         <param name="heartbeat_timeout_ms">400</param>
         <param name="startup_timeout_ms">1000</param>
-        <param name="motor_activation_interval_ms">$(arg motor_activation_interval_ms)</param>
+        <!--
+          Activation is judged from reported motor state, not from a fixed
+          delay. closed_loop_timeout_ms budgets the Heartbeat that confirms
+          Set_Axis_State took effect (Heartbeat broadcasts at ~100 ms, so
+          this tolerates several missed frames); encoder_sync_timeout_ms
+          budgets the EncoderEstimates that follow it (~10 ms each).
+          encoder_sync_frames is 2 rather than 1 deliberately. Heartbeat and
+          Get_Encoder_Estimates are independent broadcast streams, so the
+          first 0x009 seen after a closed-loop Heartbeat may have been
+          sampled by the motor before the transition the Heartbeat reports:
+          the Heartbeat itself can be up to one period old when it arrives.
+          Requiring two frames guarantees at least one estimate
+          sampled strictly after closed-loop control was already in effect,
+          which is exactly the condition that makes the position
+          trustworthy. It costs ~10 ms per joint. A larger value only adds
+          margin for hardware that skews these two streams by more than one
+          frame period, which has not been observed.
+        -->
+        <param name="closed_loop_timeout_ms">500</param>
+        <param name="encoder_sync_timeout_ms">200</param>
+        <param name="encoder_sync_frames">2</param>
         <param name="command_timeout_ms">250</param>
         <param name="scheduling_warning_ms">50</param>
