Commit message: Doc 정리 및 최신화

File: src/quattro_description/urdf/quattro.urdf.xacro (robot description, xacro)
@@ -572,16 +572,17 @@
         <param name="telemetry_period_ms">500</param>
       </hardware>
-      <xacro:quattro_hardware_joint name="front_left_hip_joint" lower="-1.04" upper="1.04"/>
-      <xacro:quattro_hardware_joint name="front_left_upper_leg_joint" lower="-1.57079632679" upper="2.59"/>
-      <xacro:quattro_hardware_joint name="front_left_lower_leg_joint" lower="-2.9" upper="1.57079632679"/>
-      <xacro:quattro_hardware_joint name="front_right_hip_joint" lower="-1.04" upper="1.04"/>
-      <xacro:quattro_hardware_joint name="front_right_upper_leg_joint" lower="-1.57079632679" upper="2.59"/>
-      <xacro:quattro_hardware_joint name="front_right_lower_leg_joint" lower="-2.9" upper="1.57079632679"/>
-      <xacro:quattro_hardware_joint name="back_left_hip_joint" lower="-1.04" upper="1.04"/>
-      <xacro:quattro_hardware_joint name="back_left_upper_leg_joint" lower="-1.57079632679" upper="2.59"/>
-      <xacro:quattro_hardware_joint name="back_left_lower_leg_joint" lower="-2.9" upper="1.57079632679"/>
-      <xacro:quattro_hardware_joint name="back_right_hip_joint" lower="-1.04" upper="1.04"/>
-      <xacro:quattro_hardware_joint name="back_right_upper_leg_joint" lower="-1.57079632679" upper="2.59"/>
-      <xacro:quattro_hardware_joint name="back_right_lower_leg_joint" lower="-2.9" upper="1.57079632679"/>
+      <!-- lower/upper mirror the <joint><limit> ranges in degrees: hip -45~45, upper -90~140, lower -135~135 -->
+      <xacro:quattro_hardware_joint name="front_left_hip_joint" lower="-0.7853981634" upper="0.7853981634"/>
+      <xacro:quattro_hardware_joint name="front_left_upper_leg_joint" lower="-1.5707963268" upper="2.4434609528"/>
+      <xacro:quattro_hardware_joint name="front_left_lower_leg_joint" lower="-2.3561944902" upper="2.3561944902"/>
+      <xacro:quattro_hardware_joint name="front_right_hip_joint" lower="-0.7853981634" upper="0.7853981634"/>
+      <xacro:quattro_hardware_joint name="front_right_upper_leg_joint" lower="-1.5707963268" upper="2.4434609528"/>
+      <xacro:quattro_hardware_joint name="front_right_lower_leg_joint" lower="-2.3561944902" upper="2.3561944902"/>
+      <xacro:quattro_hardware_joint name="back_left_hip_joint" lower="-0.7853981634" upper="0.7853981634"/>
+      <xacro:quattro_hardware_joint name="back_left_upper_leg_joint" lower="-1.5707963268" upper="2.4434609528"/>
+      <xacro:quattro_hardware_joint name="back_left_lower_leg_joint" lower="-2.3561944902" upper="2.3561944902"/>
+      <xacro:quattro_hardware_joint name="back_right_hip_joint" lower="-0.7853981634" upper="0.7853981634"/>
+      <xacro:quattro_hardware_joint name="back_right_upper_leg_joint" lower="-1.5707963268" upper="2.4434609528"/>
+      <xacro:quattro_hardware_joint name="back_right_lower_leg_joint" lower="-2.3561944902" upper="2.3561944902"/>
     </ros2_control>
   </xacro:unless>
@@ -591,16 +592,17 @@
         <plugin>gz_ros2_control/GazeboSimSystem</plugin>
       </hardware>
-      <xacro:quattro_simulation_joint name="front_left_hip_joint" lower="-1.04" upper="1.04" initial_value="0.0"/>
-      <xacro:quattro_simulation_joint name="front_left_upper_leg_joint" lower="-1.57079632679" upper="2.59" initial_value="0.63356747785"/>
-      <xacro:quattro_simulation_joint name="front_left_lower_leg_joint" lower="-2.9" upper="1.57079632679" initial_value="-1.53223802029"/>
-      <xacro:quattro_simulation_joint name="front_right_hip_joint" lower="-1.04" upper="1.04" initial_value="0.0"/>
-      <xacro:quattro_simulation_joint name="front_right_upper_leg_joint" lower="-1.57079632679" upper="2.59" initial_value="0.63356747785"/>
-      <xacro:quattro_simulation_joint name="front_right_lower_leg_joint" lower="-2.9" upper="1.57079632679" initial_value="-1.53223802029"/>
-      <xacro:quattro_simulation_joint name="back_left_hip_joint" lower="-1.04" upper="1.04" initial_value="0.0"/>
-      <xacro:quattro_simulation_joint name="back_left_upper_leg_joint" lower="-1.57079632679" upper="2.59" initial_value="0.63356747785"/>
-      <xacro:quattro_simulation_joint name="back_left_lower_leg_joint" lower="-2.9" upper="1.57079632679" initial_value="-1.53223802029"/>
-      <xacro:quattro_simulation_joint name="back_right_hip_joint" lower="-1.04" upper="1.04" initial_value="0.0"/>
-      <xacro:quattro_simulation_joint name="back_right_upper_leg_joint" lower="-1.57079632679" upper="2.59" initial_value="0.63356747785"/>
-      <xacro:quattro_simulation_joint name="back_right_lower_leg_joint" lower="-2.9" upper="1.57079632679" initial_value="-1.53223802029"/>
+      <!-- lower/upper mirror the <joint><limit> ranges in degrees: hip -45~45, upper -90~140, lower -135~135 -->
+      <xacro:quattro_simulation_joint name="front_left_hip_joint" lower="-0.7853981634" upper="0.7853981634" initial_value="0.0"/>
+      <xacro:quattro_simulation_joint name="front_left_upper_leg_joint" lower="-1.5707963268" upper="2.4434609528" initial_value="0.63356747785"/>
+      <xacro:quattro_simulation_joint name="front_left_lower_leg_joint" lower="-2.3561944902" upper="2.3561944902" initial_value="-1.53223802029"/>
+      <xacro:quattro_simulation_joint name="front_right_hip_joint" lower="-0.7853981634" upper="0.7853981634" initial_value="0.0"/>
+      <xacro:quattro_simulation_joint name="front_right_upper_leg_joint" lower="-1.5707963268" upper="2.4434609528" initial_value="0.63356747785"/>
+      <xacro:quattro_simulation_joint name="front_right_lower_leg_joint" lower="-2.3561944902" upper="2.3561944902" initial_value="-1.53223802029"/>
+      <xacro:quattro_simulation_joint name="back_left_hip_joint" lower="-0.7853981634" upper="0.7853981634" initial_value="0.0"/>
+      <xacro:quattro_simulation_joint name="back_left_upper_leg_joint" lower="-1.5707963268" upper="2.4434609528" initial_value="0.63356747785"/>
+      <xacro:quattro_simulation_joint name="back_left_lower_leg_joint" lower="-2.3561944902" upper="2.3561944902" initial_value="-1.53223802029"/>
+      <xacro:quattro_simulation_joint name="back_right_hip_joint" lower="-0.7853981634" upper="0.7853981634" initial_value="0.0"/>
+      <xacro:quattro_simulation_joint name="back_right_upper_leg_joint" lower="-1.5707963268" upper="2.4434609528" initial_value="0.63356747785"/>
+      <xacro:quattro_simulation_joint name="back_right_lower_leg_joint" lower="-2.3561944902" upper="2.3561944902" initial_value="-1.53223802029"/>
     </ros2_control>
     <gazebo>
